Commit message: Change added a Dummy Tool

File: melfa_description/urdf/rv7fl.xacro (robot description, xacro)
@@ -161,5 +161,28 @@
 	</geometry>
       </collision>
-    </link>
+      </link>
+     <joint name="jTool" type="fixed">
+      <parent link="link6"/>
+      <child link="linkTool"/>
+      <origin xyz="0 0 0.085" rpy="0 0 0"/>
+      <axis xyz="0 0 1"/>
+      <dynamics damping="0.7"/>
+      <limit upper="${360*pi/180}" lower="${-360*pi/180}" effort="10" velocity="${720*pi/180}" />
+    </joint>
+    <link name="linkTool">
+      <visual>
+	<origin rpy="0 0 0" xyz="0 0 ${-0.02/2}"/>
+	<geometry>
+      <cylinder radius="0.025" length="0.02"/>
+	</geometry>
+	<material name="white"/>
+      </visual>
+      <collision>
+	<origin rpy="0 0 0" xyz="0 0 ${-0.02/2}"/>
+	<geometry>
+	  <cylinder radius="0.025" length="0.02"/>
+	</geometry>
+      </collision>
+      </link>
   </xacro:macro>
 </robot>
